File: hdmi.kicad_sch (KiCad schematic)
At the start: 58 parts, among them J13 HDMI-Mini-C_WE_685119136923, Q1 PJE138K, Q12 PJE138K, Q2 PJE138K, Q3 PJE138K, U36 TS3DV642RUARQ1, U43 NTS0102_XSON, U44 TPD4E05U06QDQARQ1, U45 TPD4E05U06QDQARQ1, U46 TPD4E05U06QDQARQ1

Commit message: Init commit
Parts:
- C131, C132, C133, C135, C138, C139, C163, C164, C86, C87, C88, C92: LCSC Part # (none) -> C85960
- C47: LCSC Part # (none) -> C2182694
- C51: LCSC Part # (none) -> C77044
- D38: LCSC Part # (none) -> C145179
- FB4: LCSC Part # (none) -> C85840
- Q1, Q12, Q2, Q3: LCSC Part # (none) -> C391643
- R160, R211, R228, R47, R49: LCSC Part # (none) -> C202396
- R208, R227, R279, R280, R281, R282: LCSC Part # (none) -> C2076845
- R209, R210, R212, R213, R214, R220, R221, R224: LCSC Part # (none) -> C2077209
- R225, R226, R277, R278, R293, R40: LCSC Part # (none) -> C242160
- R34, R35: LCSC Part # (none) -> C1731295
- U36: LCSC Part # (none) -> C3226205
- U43: LCSC Part # (none) -> C2687851
- U44, U45, U46: LCSC Part # (none) -> C81353

Commit message: Add field Digikey Part Number. Add Chinese substitute components
Parts:
- C131, C132, C133, C135, C138, C139, C163, C164, C86, C87, C88, C92: Digikey Part # (none) -> 490-10697-1-ND
- C47: Alternative MPN (none) -> CL05A105KA5NQNC; Digikey Part # (none) -> 445-7368-1-ND
- D38: Digikey Part # (none) -> RB521S30T1GOSCT-ND
- FB4: Digikey Part # (none) -> 490-1054-1-ND
- J13: Digikey Part # (none) -> 732-2739-1-ND
- Q1, Q12, Q2, Q3: Digikey Part # (none) -> 3757-PJE138K_R1_00001CT-ND
- R160, R211, R228, R47, R49: Digikey Part # (none) -> CR0402-FX-1002GLFCT-ND
- R208, R227, R279, R280, R281, R282: Digikey Part # (none) -> CR0402-FX-2201GLFCT-ND
- R209, R210, R212, R213, R214, R220, R221, R224: Digikey Part # (none) -> CR0402-FX-4990GLFCT-ND
- R225, R226, R277, R278, R293, R40: Digikey Part # (none) -> P0.0JCT-ND
- R34, R35: Digikey Part # (none) -> Y6000CT-ND
- U36: Digikey Part # (none) -> 296-TS3DV642RUARQ1CT-ND
- U43: Digikey Part # (none) -> 568-5205-1-ND
- U44, U45, U46: Digikey Part # (none) -> 296-40696-1-ND
