File: jetson-orin-baseboard.kicad_sch (KiCad schematic)
At the start: 4 parts

Commit message: Init commit
Changed lines of the file:
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@@
 	)
 	(image
-		(at 213.36 116.84)
+		(at -81.28 137.16)
 		(scale 0.236667)
 		(data "iVBORw0KGgoAAAANSUhEUgAAB3MAAARICAYAAAAYivsYAAAABHNCSVQICAgIfAhkiAAAAAlwSFlz"
@@
 	)
 	(sheet
-		(at 203.2 203.2)
+		(at -22.86 190.5)
 		(size 12.7 12.7)
 		(fields_autoplaced yes)
@@
 		)
 		(property "Sheetname" "HDMI"
-			(at 203.2 202.4884 0)
+			(at -22.86 189.7884 0)
 			(effects
 				(font
@@
 		)
 		(property "Sheetfile" "hdmi.kicad_sch"
-			(at 203.2 216.4846 0)
+			(at -22.86 203.7846 0)
 			(effects
 				(font
@@
 	)
 	(sheet
-		(at 171.45 203.2)
+		(at -49.53 190.5)
 		(size 12.7 12.7)
 		(fields_autoplaced yes)
@@
 		)
 		(property "Sheetname" "USB3"
-			(at 171.45 202.4884 0)
+			(at -49.53 189.7884 0)
 			(effects
 				(font
@@
 		)
 		(property "Sheetfile" "usb3.kicad_sch"
-			(at 171.45 216.4846 0)
+			(at -49.53 203.7846 0)
 			(effects
 				(font
@@
 	)
 	(sheet
-		(at 171.45 228.6)
+		(at -49.53 215.9)
 		(size 12.7 12.7)
 		(fields_autoplaced yes)
@@
 		)
 		(property "Sheetname" "Supply"
-			(at 171.45 227.8884 0)
+			(at -49.53 215.1884 0)
 			(effects
 				(font
@@
 		)
 		(property "Sheetfile" "supply.kicad_sch"
-			(at 171.45 241.8846 0)
+			(at -49.53 229.1846 0)
 			(effects
 				(font
@@
 	)
 	(sheet
-		(at 76.2 203.2)
-		(size 12.7 12.7)
+		(at 195.58 73.66)
+		(size 21.59 143.51)
 		(fields_autoplaced yes)
 		(stroke
-			(width 0.1524)
+			(width 0.3048)
 			(type solid)
+			(color 0 0 255 1)
 		)
 		(fill
@@
 		)
 		(property "Sheetname" "SoM"
-			(at 76.2 202.4884 0)
+			(at 195.58 70.9672 0)
 			(effects
 				(font
-					(size 1.27 1.27)
+					(face "ISOCPEUR")
+					(size 5.08 5.08)
+					(bold yes)
 				)
 				(justify left bottom)
@@
 		)
 		(property "Sheetfile" "som.kicad_sch"
-			(at 76.2 216.4846 0)
+			(at 195.58 217.8308 0)
 			(effects
 				(font
@@
 	)
 	(sheet
-		(at 107.95 228.6)
+		(at -113.03 215.9)
 		(size 12.7 12.7)
 		(fields_autoplaced yes)
@@
 		)
 		(property "Sheetname" "CSI"
-			(at 107.95 227.8884 0)
+			(at -113.03 215.1884 0)
 			(effects
 				(font
@@
 		)
 		(property "Sheetfile" "csi.kicad_sch"
-			(at 107.95 241.8846 0)
+			(at -113.03 229.1846 0)
 			(effects
 				(font
@@
 	)
 	(sheet
-		(at 107.95 203.2)
+		(at -113.03 190.5)
 		(size 12.7 12.7)
 		(fields_autoplaced yes)
@@
 		)
 		(property "Sheetname" "M.2"
-			(at 107.95 202.4884 0)
+			(at -113.03 189.7884 0)
 			(effects
 				(font
@@
 		)
 		(property "Sheetfile" "m-2.kicad_sch"
-			(at 107.95 216.4846 0)
+			(at -113.03 203.7846 0)
 			(effects
 				(font
@@
 	)
 	(sheet
-		(at 76.2 228.6)
+		(at -144.78 215.9)
 		(size 12.7 12.7)
 		(fields_autoplaced yes)
@@
 		)
 		(property "Sheetname" "Ethernet"
-			(at 76.2 227.8884 0)
+			(at -144.78 215.1884 0)
 			(effects
 				(font
@@
 		)
 		(property "Sheetfile" "ethernet.kicad_sch"
-			(at 76.2 241.8846 0)
+			(at -144.78 229.1846 0)
 			(effects
 				(font
@@
 	)
 	(sheet
-		(at 139.7 228.6)
+		(at -81.28 215.9)
 		(size 12.7 12.7)
 		(fields_autoplaced yes)
@@
 		)
 		(property "Sheetname" "Peripherals"
-			(at 139.7 227.8884 0)
+			(at -81.28 215.1884 0)
 			(effects
 				(font
@@
 		)
 		(property "Sheetfile" "peripherals.kicad_sch"
-			(at 139.7 241.8846 0)
+			(at -81.28 229.1846 0)
 			(effects
 				(font
@@
 	)
 	(sheet
-		(at 139.7 203.2)
+		(at -81.28 190.5)
 		(size 12.7 12.7)
 		(fields_autoplaced yes)
@@
 		)
 		(property "Sheetname" "USB Debug, DP"
-			(at 139.7 202.4884 0)
+			(at -81.28 189.7884 0)
 			(effects
 				(font
@@
 		)
 		(property "Sheetfile" "usb.kicad_sch"
-			(at 139.7 216.4846 0)
+			(at -81.28 203.7846 0)
 			(effects
 				(font

Commit message: Add field Digikey Part Number. Add Chinese substitute components
Parts:
- H3, H4, H5, H6: Digikey Part # (none) -> 732-9774065151RCT-ND
Other:
- note added: "+-------------------+----------+ | Section | Page No.| +-------------------+----------+ | SoM | 2 | M.2 | 3 | USB Debug, DP | 4 | USB3 | 5 | HDMI connector | 6 | Ethernet | 7 | CSI | 8 | Peripherals | 9 | Supply | 10 +-------------------+----------+"
- note added: "Sustitute to H1...H7: SMTWE2565MTJ (Chinese brand)"
- note added: "github.com/antmicro/jetson-orin-baseboard https://antmicro.github.io/jetson-orin-baseboard/getting_started.html#"
- note removed: "github.com/antmicro/jetson-orin-baseboard"
Changed lines of the file:
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@@
 		)
 	)
-	(text "github.com/antmicro/jetson-orin-baseboard"
+	(text "github.com/antmicro/jetson-orin-baseboard\nhttps://antmicro.github.io/jetson-orin-baseboard/getting_started.html#"
 		(exclude_from_sim no)
-		(at 14.605 31.115 0)
+		(at 14.732 35.052 0)
 		(effects
 			(font
@@
 			)
 			(justify left bottom)
+		)
+	)
+	(text "Sustitute to H1...H7:\nSMTWE2565MTJ (Chinese brand)"
+		(exclude_from_sim no)
+		(at 365.506 246.126 0)
+		(effects
+			(font
+				(size 1.27 1.27)
+			)
+			(justify left)
+		)
+	)
+	(text "+-------------------+----------+\n|      Section      |  Page No.|\n+-------------------+----------+\n| SoM               |    2     \n| M.2                |    3     \n| USB Debug, DP     |    4     \n| USB3              |    5     \n| HDMI connector    |    6     \n| Ethernet          |    7     \n| CSI               |    8     \n| Peripherals       |    9     \n| Supply            |   10     \n+-------------------+----------+\n"
+		(exclude_from_sim no)
+		(at 382.016 125.984 0)
+		(effects
+			(font
+				(size 2.54 2.54)
+			)
+			(justify right)
 		)
 	)
@@
 			)
 		)
+		(property "Digikey Part #" "732-9774065151RCT-ND"
+			(at 368.3 215.9 0)
+			(effects
+				(font
+					(size 1.27 1.27)
+				)
+				(hide yes)
+			)
+		)
 		(pin "1"
 		)
@@
 			)
 		)
+		(property "Digikey Part #" "732-9774065151RCT-ND"
+			(at 368.3 228.6 0)
+			(effects
+				(font
+					(size 1.27 1.27)
+				)
+				(hide yes)
+			)
+		)
 		(pin "1"
 		)
@@
 			)
 		)
+		(property "Digikey Part #" "732-9774065151RCT-ND"
+			(at 368.3 222.25 0)
+			(effects
+				(font
+					(size 1.27 1.27)
+				)
+				(hide yes)
+			)
+		)
 		(pin "1"
 		)
@@
 			)
 		)
+		(property "Digikey Part #" "732-9774065151RCT-ND"
+			(at 368.3 234.95 0)
+			(effects
+				(font
+					(size 1.27 1.27)
+				)
+				(hide yes)
+			)
+		)
 		(pin "1"
 		)
@@
 	)
 	(sheet
-		(at -22.86 190.5)
+		(at 143.51 185.42)
 		(size 12.7 12.7)
 		(fields_autoplaced yes)
@@
 		)
 		(property "Sheetname" "HDMI"
-			(at -22.86 189.7884 0)
+			(at 143.51 184.7084 0)
 			(effects
 				(font
@@
 		)
 		(property "Sheetfile" "hdmi.kicad_sch"
-			(at -22.86 203.7846 0)
+			(at 143.51 198.7046 0)
 			(effects
 				(font
@@
 	)
 	(sheet
-		(at -49.53 190.5)
+		(at 143.51 113.03)
 		(size 12.7 12.7)
 		(fields_autoplaced yes)
@@
 		)
 		(property "Sheetname" "USB3"
-			(at -49.53 189.7884 0)
+			(at 143.51 112.3184 0)
 			(effects
 				(font
@@
 		)
 		(property "Sheetfile" "usb3.kicad_sch"
-			(at -49.53 203.7846 0)
+			(at 143.51 126.3146 0)
 			(effects
 				(font
@@
 	)
 	(sheet
-		(at -49.53 215.9)
+		(at 118.11 44.45)
 		(size 12.7 12.7)
 		(fields_autoplaced yes)
@@
 		)
 		(property "Sheetname" "Supply"
-			(at -49.53 215.1884 0)
+			(at 118.11 43.7384 0)
 			(effects
 				(font
@@
 		)
 		(property "Sheetfile" "supply.kicad_sch"
-			(at -49.53 229.1846 0)
+			(at 118.11 57.7346 0)
 			(effects
 				(font
@@
 	)
 	(sheet
-		(at 195.58 73.66)
+		(at 71.12 69.85)
 		(size 21.59 143.51)
 		(fields_autoplaced yes)
@@
 		)
 		(property "Sheetname" "SoM"
-			(at 195.58 70.9672 0)
+			(at 71.12 67.1572 0)
 			(effects
 				(font
@@
 		)
 		(property "Sheetfile" "som.kicad_sch"
-			(at 195.58 217.8308 0)
+			(at 71.12 214.0208 0)
 			(effects
 				(font
@@
 	)
 	(sheet
-		(at -113.03 215.9)
+		(at 143.51 162.56)
 		(size 12.7 12.7)
 		(fields_autoplaced yes)
@@
 		)
 		(property "Sheetname" "CSI"
-			(at -113.03 215.1884 0)
+			(at 143.51 161.8484 0)
 			(effects
 				(font
@@
 		)
 		(property "Sheetfile" "csi.kicad_sch"
-			(at -113.03 229.1846 0)
+			(at 143.51 175.8446 0)
 			(effects
 				(font
@@
 	)
 	(sheet
-		(at -113.03 190.5)
+		(at 143.51 67.31)
 		(size 12.7 12.7)
 		(fields_autoplaced yes)
@@
 		)
 		(property "Sheetname" "M.2"
-			(at -113.03 189.7884 0)
+			(at 143.51 66.5984 0)
 			(effects
 				(font
@@
 		)
 		(property "Sheetfile" "m-2.kicad_sch"
-			(at -113.03 203.7846 0)
+			(at 143.51 80.5946 0)
 			(effects
 				(font
@@
 	)
 	(sheet
-		(at -144.78 215.9)
+		(at 143.51 139.7)
 		(size 12.7 12.7)
 		(fields_autoplaced yes)
@@
 		)
 		(property "Sheetname" "Ethernet"
-			(at -144.78 215.1884 0)
+			(at 143.51 138.9884 0)
 			(effects
 				(font
@@
 		)
 		(property "Sheetfile" "ethernet.kicad_sch"
-			(at -144.78 229.1846 0)
+			(at 143.51 152.9846 0)
 			(effects
 				(font
@@
 	)
 	(sheet
-		(at -81.28 215.9)
+		(at 143.51 209.55)
 		(size 12.7 12.7)
 		(fields_autoplaced yes)
@@
 		)
 		(property "Sheetname" "Peripherals"
-			(at -81.28 215.1884 0)
+			(at 143.51 208.8384 0)
 			(effects
 				(font
@@
 		)
 		(property "Sheetfile" "peripherals.kicad_sch"
-			(at -81.28 229.1846 0)
+			(at 143.51 222.8346 0)
 			(effects
 				(font
@@
 	)
 	(sheet
-		(at -81.28 190.5)
+		(at 143.51 90.17)
 		(size 12.7 12.7)
 		(fields_autoplaced yes)
@@
 		)
 		(property "Sheetname" "USB Debug, DP"
-			(at -81.28 189.7884 0)
+			(at 143.51 89.4584 0)
 			(effects
 				(font
@@
 		)
 		(property "Sheetfile" "usb.kicad_sch"
-			(at -81.28 203.7846 0)
-			(effects
-				(font
+			(at 143.51 103.4546 0)
+			(effects
+				(font

Commit message: Update: reorganized schematic layout for Jetson Orin Baseboard
Other:
- note added: "Created by:"
- note added: "Modified and manufactured by:"
- note removed: "+-------------------+----------+ | Section | Page No.| +-------------------+----------+ | SoM | 2 | M.2 | 3 | USB Debug, DP | 4 | USB3 | 5 | HDMI connector | 6 | Ethernet | 7 | CSI | 8 | Peripherals | 9 | Supply | 10 +-------------------+----------+"
- note removed: "github.com/antmicro/jetson-orin-baseboard https://antmicro.github.io/jetson-orin-baseboard/getting_started.html#"
- moved on the sheet: H3, H4, H5, H6
