File: m-2.kicad_sch (KiCad schematic)
At the start: 61 parts, among them J1 Bus_M.2_2199230-6, J2 Bus_M.2_1-2199230-6, M3 Mech_M2_2280_H2.5mm, U2 74LVC2G07_SOT457, U3 74LVC2G07_SOT457, Y1 Oscillator_32.768kHz_ECS_2520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

Commit message: Init commit
Parts:
- C10, C13, C14, C15, C16, C17, C18, C19, C20, C9: LCSC Part # (none) -> C106257
- C11, C12, C21, C22, C23, C24: LCSC Part # (none) -> C77044
- C25, C7, C8: LCSC Part # (none) -> C85960
- D1, D51, D52: LCSC Part # (none) -> C125093
- J1, J2: LCSC Part # (none) -> C4710843
- R13, R14, R15, R16, R17, R18, R19, R20, R29, R30, R31, R52: LCSC Part # (none) -> C242160
- R143: LCSC Part # (none) -> C253507
- R186, R187, R39: LCSC Part # (none) -> C19946422
- R21, R22: LCSC Part # (none) -> C1731295
- R27, R28, R32, R37, R38: LCSC Part # (none) -> C2091678
- U2, U3: LCSC Part # (none) -> C548568
- Y1: LCSC Part # (none) -> C5375606

Commit message: Add field Digikey Part Number. Add Chinese substitute components
Parts:
- C10, C13, C14, C15, C16, C17, C18, C19, C20, C9: Digikey Part # (none) -> 311-1421-1-ND
- C25, C7, C8: Digikey Part # (none) -> 490-10697-1-ND
- D1, D51, D52: Alternative MPN (none) -> LTST-C190KRKT; Digikey Part # (none) -> 160-1183-1-ND
- J2: Digikey Part # (none) -> A118046CT-ND
- R13, R14, R15, R16, R17, R18, R19, R20, R29, R30, R31, R52: Digikey Part # (none) -> P0.0JCT-ND
- R143: Digikey Part # (none) -> 846-PMR03EZPJ000CT-ND
- R186, R187, R39: Digikey Part # (none) -> CR0402-FX-2000GLFCT-ND
- R21, R22: Digikey Part # (none) -> Y6000CT-ND
- R27, R28, R32, R37, R38: Digikey Part # (none) -> CR0402-FX-4702GLFCT-ND
- SP7, SP8: Digikey Part # (none) -> 732-7078-1-ND
- U2, U3: Digikey Part # (none) -> 1727-6087-1-ND
- Y1: Digikey Part # (none) -> 50-ECS-327MVATX-2-CN-TR3CT-ND
