File: usb3.kicad_sch (KiCad schematic)
At the start: 51 parts, among them J5 USB-C_WE_632723300011, Q19 PJE138K, Q4 PJE138K, U17 HD3SS3220RNH, U18 AP22615A_TSOT26, U19 TPD4E05U06QDQARQ1, U20 TPD4E05U06QDQARQ1, U21 TPD4E05U06QDQARQ1

Commit message: Init commit
Parts:
- C66, C74: LCSC Part # (none) -> C77044
- C67, C68, C69, C70, C71, C72, C73, C75: LCSC Part # (none) -> C85960
- D10: LCSC Part # (none) -> C41364466
- D11: LCSC Part # (none) -> C125093
- Q19, Q4: LCSC Part # (none) -> C391643
- R113, R114, R118, R119, R124, R125, R200, R201, R202, R203, R23, R245: LCSC Part # (none) -> C242160
- R115, R116, R135, R136, R137, R138, R24, R60: LCSC Part # (none) -> C202396
- R126, R265, R266, R61: LCSC Part # (none) -> C2077217
- R128: LCSC Part # (none) -> C409935
- R139: LCSC Part # (none) -> C2076845
- R140: LCSC Part # (none) -> C2077077
- R184: LCSC Part # (none) -> C202394
- U17: LCSC Part # (none) -> C2155924
- U18: LCSC Part # (none) -> C2680357
- U19, U20, U21: LCSC Part # (none) -> C81353

Commit message: Add field Digikey Part Number. Add Chinese substitute components
Parts:
- C67, C68, C69, C70, C71, C72, C73, C75: Digikey Part # (none) -> 490-10697-1-ND
- D10: Digikey Part # (none) -> ESD9X5.0ST5GOSCT-ND
- D11: Alternative MPN (none) -> LTST-C190KRKT; Digikey Part # (none) -> 160-1183-1-ND
- J5: Digikey Part # (none) -> 732-9618-1-ND
- Q19, Q4: Digikey Part # (none) -> 3757-PJE138K_R1_00001CT-ND
- R113, R114, R118, R119, R124, R125, R200, R201, R202, R203, R23, R245: Digikey Part # (none) -> P0.0JCT-ND
- R115, R116, R135, R136, R137, R138, R24, R60: Digikey Part # (none) -> CR0402-FX-1002GLFCT-ND
- R126, R265, R266, R61: Digikey Part # (none) -> CR0402-FX-2003GLFCT-ND
- R128: Digikey Part # (none) -> P887KLCT-ND
- R139: Digikey Part # (none) -> CR0402-FX-2201GLFCT-ND
- R140: Digikey Part # (none) -> CR0402-FX-4700GLFCT-ND
- R184: Digikey Part # (none) -> CR0402-FX-1001GLFCT-ND
- U17: Digikey Part # (none) -> 296-49643-1-ND
- U18: Digikey Part # (none) -> AP22615AWU-7DICT-ND
- U19, U20, U21: Digikey Part # (none) -> 296-40696-1-ND

Commit message: Update: reorganized schematic layout for Jetson Orin Baseboard
Changed lines of the file:
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@@
 (kicad_sch
-	(version 20231120)
+	(version 20250114)
 	(generator "eeschema")
-	(generator_version "8.0")
+	(generator_version "9.0")
 	(paper "A3")
 	(title_block
@@
 		(comment 1 "www.antmicro.com")
 	)
+	(text "Mode\nHIGH - DFP (HOST ONLY)\nLOW  - UFP (DEVICE ONLY)\nDNP  - DRP (DUAL ROLE PORT)\n"
+		(exclude_from_sim no)
+		(at 72.39 132.715 0)
+		(effects
+			(font
+				(size 1.27 1.27)
+			)
+			(justify left bottom)
+		)
+	)
+	(text "Enable MUX"
+		(exclude_from_sim no)
+		(at 99.695 139.7 0)
+		(effects
+			(font
+				(size 1.27 1.27)
+			)
+			(justify left bottom)
+		)
+	)
+	(text "Both DNP - GPIO Mode\nHIGH - I2C Mode 0x67\nLOW -  I2C Mode 0x47"
+		(exclude_from_sim no)
+		(at 50.165 184.785 0)
+		(effects
+			(font
+				(size 1.27 1.27)
+			)
+			(justify left bottom)
+		)
+	)
+	(text "USB-C 1"
+		(exclude_from_sim no)
+		(at 195.58 58.42 0)
+		(effects
+			(font
+				(size 4 4)
+				(thickness 0.8)
+				(bold yes)
+			)
+			(justify left bottom)
+		)
+	)
+	(text "10k - 3A\n500k - 1.5A\nDNP - 900mA"
+		(exclude_from_sim no)
+		(at 128.905 132.08 0)
+		(effects
+			(font
+				(size 1.27 1.27)
+			)
+			(justify left bottom)
+		)
+	)
+	(text "LOW: DFP role \nHIGH: NO ATTACH/UFP"
+		(exclude_from_sim no)
+		(at 222.25 121.92 0)
+		(effects
+			(font
+				(size 1.27 1.27)
+			)
+			(justify left bottom)
+		)
+	)
+	(text "NOTE:\nPopulate 1/3"
+		(exclude_from_sim no)
+		(at 325.755 62.865 0)
+		(effects
+			(font
+				(size 1.27 1.27)
+			)
+			(justify left bottom)
+		)
+	)
+	(text "USBC1"
+		(exclude_from_sim no)
+		(at 305.435 129.54 0)
+		(effects
+			(font
+				(size 1.27 1.27)
+				(thickness 0.254)
+				(bold yes)
+			)
+			(justify left bottom)
+		)
+	)
+	(text "LOW: VCONN OC TRIP \nHIGH: NORMAL OPERATION"
+		(exclude_from_sim no)
+		(at 222.25 128.27 0)
+		(effects
+			(font
+				(size 1.27 1.27)
+			)
+			(justify left bottom)
+		)
+	)
+	(text "Enable CC controller"
+		(exclude_from_sim no)
+		(at 90.805 142.24 0)
+		(effects
+			(font
+				(size 1.27 1.27)
+			)
+			(justify left bottom)
+		)
+	)
 	(junction
 		(at 213.36 90.17)
@@
 		)
 	)
-	(text "Mode\nHIGH - DFP (HOST ONLY)\nLOW  - UFP (DEVICE ONLY)\nDNP  - DRP (DUAL ROLE PORT)\n"
-		(exclude_from_sim no)
-		(at 72.39 132.715 0)
-		(effects
-			(font
-				(size 1.27 1.27)
-			)
-			(justify left bottom)
-		)
-	)
-	(text "Enable MUX"
-		(exclude_from_sim no)
-		(at 99.695 139.7 0)
-		(effects
-			(font
-				(size 1.27 1.27)
-			)
-			(justify left bottom)
-		)
-	)
-	(text "Both DNP - GPIO Mode\nHIGH - I2C Mode 0x67\nLOW -  I2C Mode 0x47"
-		(exclude_from_sim no)
-		(at 50.165 184.785 0)
-		(effects
-			(font
-				(size 1.27 1.27)
-			)
-			(justify left bottom)
-		)
-	)
-	(text "USB-C 1"
-		(exclude_from_sim no)
-		(at 195.58 58.42 0)
-		(effects
-			(font
-				(size 4 4)
-				(thickness 0.8)
-				(bold yes)
-			)
-			(justify left bottom)
-		)
-	)
-	(text "10k - 3A\n500k - 1.5A\nDNP - 900mA"
-		(exclude_from_sim no)
-		(at 128.905 132.08 0)
-		(effects
-			(font
-				(size 1.27 1.27)
-			)
-			(justify left bottom)
-		)
-	)
-	(text "LOW: DFP role \nHIGH: NO ATTACH/UFP"
-		(exclude_from_sim no)
-		(at 222.25 121.92 0)
-		(effects
-			(font
-				(size 1.27 1.27)
-			)
-			(justify left bottom)
-		)
-	)
-	(text "NOTE:\nPopulate 1/3"
-		(exclude_from_sim no)
-		(at 325.755 62.865 0)
-		(effects
-			(font
-				(size 1.27 1.27)
-			)
-			(justify left bottom)
-		)
-	)
-	(text "USBC1"
-		(exclude_from_sim no)
-		(at 305.435 129.54 0)
-		(effects
-			(font
-				(size 1.27 1.27)
-				(thickness 0.254)
-				(bold yes)
-			)
-			(justify left bottom)
-		)
-	)
-	(text "LOW: VCONN OC TRIP \nHIGH: NORMAL OPERATION"
-		(exclude_from_sim no)
-		(at 222.25 128.27 0)
-		(effects
-			(font
-				(size 1.27 1.27)
-			)
-			(justify left bottom)
-		)
-	)
-	(text "Enable CC controller"
-		(exclude_from_sim no)
-		(at 90.805 142.24 0)
-		(effects
-			(font
-				(size 1.27 1.27)
-			)
-			(justify left bottom)
-		)
-	)
